File: schematics/Thermostat_WKR.kicad_sch (KiCad schematic)
At the start: 10 parts, among them J1 Dupont 6pin, J2 Dupont 6pin, SW1 Button Down, SW2 Button Up, SW3 Button Enter

Commit message: commit
Connections:
- net at A1.4 (SDA), U1.33 (SDA/V_SPI_HD/GPIO21): now also J2.4 (Pin_4); no longer J2.5 (Pin_5)
- net at A1.3 (SCK), U1.36 (SCL/V_SPI_WP/GPIO22): now also J2.5 (Pin_5); no longer J2.4 (Pin_4)
- net at U3.3 (SCL): now also J1.5 (Pin_5); no longer J1.4 (Pin_4)
- net at U3.4 (SDA): now also J1.4 (Pin_4); no longer J1.5 (Pin_5)
Other:
- note added: "5V GND 3.3V SDA SCL spare"
- note removed: "5V GND 3.3V SCL SDA spare"
Changed lines of the file:
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@@
 		(rev "0")
 	)
-	(text "5V\nGND\n3.3V\nSCL\nSDA\nspare"
+	(text "5V\nGND\n3.3V\nSDA\nSCL\nspare"
 		(exclude_from_sim no)
 		(at 127 66.294 0)
@@
 	)
 	(junction
-		(at 154.94 69.85)
-		(diameter 0)
-		(color 0 0 0 0)
-	)
-	(junction
-		(at 152.4 67.31)
-		(diameter 0)
-		(color 0 0 0 0)
-	)
-	(junction
 		(at 93.98 63.5)
 		(diameter 0)
@@
 	)
 	(junction
+		(at 154.94 67.31)
+		(diameter 0)
+		(color 0 0 0 0)
+	)
+	(junction
 		(at 154.94 110.49)
 		(diameter 0)
@@
 	)
 	(junction
+		(at 152.4 69.85)
+		(diameter 0)
+		(color 0 0 0 0)
+	)
+	(junction
 		(at 147.32 59.69)
 		(diameter 0)
@@
 		(color 0 0 0 0)
 	)
+	(junction
+		(at 154.94 52.07)
+		(diameter 0)
+		(color 0 0 0 0)
+	)
 	(wire
 		(pts
@@
 	(wire
 		(pts
-			(xy 135.89 69.85) (xy 154.94 69.85)
+			(xy 135.89 69.85) (xy 152.4 69.85)
 		)
 		(stroke
@@
 	(wire
 		(pts
+			(xy 154.94 67.31) (xy 228.6 67.31)
+		)
+		(stroke
+			(width 0)
+			(type default)
+		)
+	)
+	(wire
+		(pts
 			(xy 167.64 101.6) (xy 168.91 101.6)
 		)
@@
 	(wire
 		(pts
+			(xy 109.22 67.31) (xy 118.11 67.31)
+		)
+		(stroke
+			(width 0)
+			(type default)
+		)
+	)
+	(wire
+		(pts
 			(xy 176.53 118.11) (xy 154.94 118.11)
 		)
@@
 	(wire
 		(pts
-			(xy 228.6 69.85) (xy 154.94 69.85)
-		)
-		(stroke
-			(width 0)
-			(type default)
-		)
-	)
-	(wire
-		(pts
 			(xy 135.89 59.69) (xy 147.32 59.69)
 		)
@@
 	(wire
 		(pts
-			(xy 152.4 67.31) (xy 152.4 52.07)
-		)
-		(stroke
-			(width 0)
-			(type default)
-		)
-	)
-	(wire
-		(pts
 			(xy 157.48 110.49) (xy 154.94 110.49)
 		)
@@
 	(wire
 		(pts
+			(xy 228.6 67.31) (xy 228.6 97.79)
+		)
+		(stroke
+			(width 0)
+			(type default)
+		)
+	)
+	(wire
+		(pts
 			(xy 173.99 64.77) (xy 135.89 64.77)
 		)
@@
 	(wire
 		(pts
+			(xy 226.06 90.17) (xy 219.71 90.17)
+		)
+		(stroke
+			(width 0)
+			(type default)
+		)
+	)
+	(wire
+		(pts
 			(xy 135.89 62.23) (xy 149.86 62.23)
 		)
@@
 	(wire
 		(pts
-			(xy 228.6 97.79) (xy 228.6 69.85)
-		)
-		(stroke
-			(width 0)
-			(type default)
-		)
-	)
-	(wire
-		(pts
-			(xy 226.06 90.17) (xy 226.06 67.31)
-		)
-		(stroke
-			(width 0)
-			(type default)
-		)
-	)
-	(wire
-		(pts
-			(xy 106.68 105.41) (xy 106.68 67.31)
+			(xy 226.06 69.85) (xy 226.06 90.17)
 		)
 		(stroke
@@
 	(wire
 		(pts
-			(xy 106.68 67.31) (xy 118.11 67.31)
+			(xy 154.94 49.53) (xy 154.94 52.07)
 		)
 		(stroke
@@
 	(wire
 		(pts
-			(xy 109.22 69.85) (xy 118.11 69.85)
+			(xy 106.68 69.85) (xy 118.11 69.85)
 		)
 		(stroke
@@
 	(wire
 		(pts
-			(xy 154.94 69.85) (xy 154.94 52.07)
-		)
-		(stroke
-			(width 0)
-			(type default)
-		)
-	)
-	(wire
-		(pts
-			(xy 219.71 90.17) (xy 226.06 90.17)
+			(xy 228.6 97.79) (xy 219.71 97.79)
+		)
+		(stroke
+			(width 0)
+			(type default)
+		)
+	)
+	(wire
+		(pts
+			(xy 154.94 67.31) (xy 154.94 52.07)
 		)
 		(stroke
@@
 	(wire
 		(pts
-			(xy 135.89 67.31) (xy 152.4 67.31)
+			(xy 109.22 67.31) (xy 109.22 107.95)
 		)
 		(stroke
@@
 	(wire
 		(pts
-			(xy 226.06 67.31) (xy 152.4 67.31)
+			(xy 152.4 69.85) (xy 226.06 69.85)
+		)
+		(stroke
+			(width 0)
+			(type default)
+		)
+	)
+	(wire
+		(pts
+			(xy 135.89 67.31) (xy 154.94 67.31)
 		)
 		(stroke
@@
 	(wire
 		(pts
+			(xy 106.68 69.85) (xy 106.68 105.41)
+		)
+		(stroke
+			(width 0)
+			(type default)
+		)
+	)
+	(wire
+		(pts
 			(xy 96.52 64.77) (xy 118.11 64.77)
 		)
@@
 	(wire
 		(pts
-			(xy 219.71 97.79) (xy 228.6 97.79)
-		)
-		(stroke
-			(width 0)
-			(type default)
-		)
-	)
-	(wire
-		(pts
 			(xy 82.55 100.33) (xy 96.52 100.33)
 		)
@@
 	(wire
 		(pts
-			(xy 109.22 107.95) (xy 109.22 69.85)
-		)
-		(stroke
-			(width 0)
-			(type default)
-		)
-	)
-	(wire
-		(pts
 			(xy 154.94 110.49) (xy 154.94 101.6)
 		)
@@
 		)
 		(stroke
+			(width 0)
+			(type default)
+		)
+	)
+	(wire
+		(pts
+			(xy 152.4 52.07) (xy 152.4 69.85)
+		)
+		(stroke
